File: kicad/hive/beehive-hive.kicad_sch (KiCad schematic)
At the start: 0 parts

Commit message: feat: draw the hive board schematic
SHT40-AD1F and ICS-43434 with decoupling, the SD pull-down and an RJ45 jack whose pinout puts each clock on a T568 pair with a ground. Test points on every net; every part carries its LCSC number.
Parts:
- added C1, C2: 100n, Capacitor_SMD:C_0603_1608Metric, symbol Device:C
- added C3: 10u, Capacitor_SMD:C_0603_1608Metric, symbol Device:C
- added H1, H2: MountingHole, MountingHole:MountingHole_3.2mm_M3, symbol Mechanical:MountingHole
- added J1: RJHSE5380, Connector_RJ:RJ45_Amphenol_RJHSE5380, symbol Connector:RJ45_Shielded
- added MK1: ICS-43434, Sensor_Audio:InvenSense_ICS-43434-6_3.5x2.65mm, symbol Sensor_Audio:ICS-43434
- added R1: 100k, Resistor_SMD:R_0603_1608Metric, symbol Device:R
- added TP1: 3V3, TestPoint:TestPoint_Pad_D1.5mm, symbol Connector:TestPoint
- added TP2: GND, TestPoint:TestPoint_Pad_D1.5mm, symbol Connector:TestPoint
- added TP3: SDA, TestPoint:TestPoint_Pad_D1.5mm, symbol Connector:TestPoint
- added TP4: SCL, TestPoint:TestPoint_Pad_D1.5mm, symbol Connector:TestPoint
- added TP5: WS, TestPoint:TestPoint_Pad_D1.5mm, symbol Connector:TestPoint
- added TP6: SCK, TestPoint:TestPoint_Pad_D1.5mm, symbol Connector:TestPoint
- added TP7: SD, TestPoint:TestPoint_Pad_D1.5mm, symbol Connector:TestPoint
- added U1: SHT40-AD1F, Sensor_Humidity:Sensirion_DFN-4_1.5x1.5mm_P0.8mm_SHT4x_NoCentralPad, symbol Sensor_Humidity:SHT4x
Connections:
- new net +3V3: C1.1, C2.1, C3.1, J1.5, MK1.5 (VDD), TP1.1, U1.3 (VDD)
- new net GND: C1.2, C2.2, C3.2, J1.2, J1.6, J1.SH, MK1.2 (LR), MK1.3 (GND), R1.2, TP2.1, U1.4 (VSS)
- new net SCK: J1.1, MK1.4 (SCK), TP6.1
- new net SCL: J1.3, TP4.1, U1.2 (SCL)
- new net SD: J1.8, MK1.6 (SD), R1.1, TP7.1
- new net SDA: J1.4, TP3.1, U1.1 (SDA)
- new net WS: J1.7, MK1.1 (WS), TP5.1

Commit message: fix: act on the schematic review
The I2C pull-ups move to the Feather's always-on 3V3 so they no longer
feed the sensor rail during deep sleep. Both boards get SRV05-4 ESD
arrays on every hive cable line, with VP open so the steering diodes
cannot back-power the rail either. The microphone drives the cable
through 33 Ω, the charger input capacitor is now 25 V, and the battery
connector's value names its polarity.
Parts:
- added R2: 33, Resistor_SMD:R_0603_1608Metric, symbol Device:R
- added U2, U3: SRV05-4, Package_TO_SOT_SMD:SOT-23-6, symbol Power_Protection:SRV05-4
Connections:
- net +3V3: now also U3.3 (IO2)
- net GND: now also U2.2 (VN), U3.2 (VN)
- net SCK: now also U2.6 (IO4)
- net SCL: now also U2.3 (IO2)
- net SD: now also R2.2, U3.1 (IO1); no longer MK1.6 (SD)
- net SDA: now also U2.1 (IO1)
- net WS: now also U2.4 (IO3)
- new net SD_MK: MK1.6 (SD), R2.1
- no-connect marks 0 -> 4
