File: kicad/hive/beehive-hive.kicad_pcb (KiCad board)
At the start: 2 copper layers, 0 parts

Commit message: feat: place and route the hive board
GND pours on both layers, stitched so every top-layer fragment reaches ground.
Parts:
- added C1: 100n, Capacitor_SMD:C_0603_1608Metric, F.Cu at (119.5, 124.5)
- added C2: 100n, Capacitor_SMD:C_0603_1608Metric, F.Cu at (110.9, 125.2)
- added C3: 10u, Capacitor_SMD:C_0603_1608Metric, F.Cu at (118.5, 120.0)
- added H1: MountingHole, MountingHole:MountingHole_3.2mm_M3, F.Cu at (103.5, 136.5)
- added H2: MountingHole, MountingHole:MountingHole_3.2mm_M3, F.Cu at (120.5, 136.5)
- added J1: RJHSE5380, Connector_RJ:RJ45_Amphenol_RJHSE5380, F.Cu at (106.5, 108.2)
- added MK1: ICS-43434, Sensor_Audio:InvenSense_ICS-43434-6_3.5x2.65mm, F.Cu at (108.0, 126.5)
- added R1: 100k, Resistor_SMD:R_0603_1608Metric, F.Cu at (112.5, 130.5)
- added R2: 33, Resistor_SMD:R_0603_1608Metric, F.Cu at (108.0, 130.0)
- added TP1: 3V3, TestPoint:TestPoint_Pad_D1.5mm, F.Cu at (108.5, 133.5)
- added TP2: GND, TestPoint:TestPoint_Pad_D1.5mm, F.Cu at (111.0, 133.5)
- added TP3: SDA, TestPoint:TestPoint_Pad_D1.5mm, F.Cu at (113.6, 133.5)
- added TP4: SCL, TestPoint:TestPoint_Pad_D1.5mm, F.Cu at (108.5, 136.0)
- added TP5: WS, TestPoint:TestPoint_Pad_D1.5mm, F.Cu at (111.0, 136.0)
- added TP6: SCK, TestPoint:TestPoint_Pad_D1.5mm, F.Cu at (113.6, 136.0)
- added TP7: SD, TestPoint:TestPoint_Pad_D1.5mm, F.Cu at (108.5, 138.5)
- added U1: SHT40-AD1F, Sensor_Humidity:Sensirion_DFN-4_1.5x1.5mm_P0.8mm_SHT4x_NoCentralPad, F.Cu at (119.5, 128.0)
- added U2: SRV05-4, Package_TO_SOT_SMD:SOT-23-6, F.Cu at (105.0, 120.0)
- added U3: SRV05-4, Package_TO_SOT_SMD:SOT-23-6, F.Cu at (111.5, 120.0)
Routing:
- net /+3V3: track 0.00 -> 62.3 mm
- net /SDA: track 0.00 -> 49.1 mm, vias 0 -> 2
- net /SCL: track 0.00 -> 44.9 mm
- net /SD: track 0.00 -> 38.1 mm, vias 0 -> 2
- net /WS: track 0.00 -> 35.9 mm, vias 0 -> 2
- net /SCK: track 0.00 -> 34.8 mm, vias 0 -> 3
- net /SD_MK: track 0.00 -> 7.27 mm, vias 0 -> 2
- net /GND: track 0.00 -> 3.05 mm, vias 0 -> 7
- added copper zone on B.Cu, net /GND
- added copper zone on F.Cu, net /GND
Other:
- board outline added: 24 x 40 mm
