File: kicad/main/beehive-main.kicad_sch (KiCad schematic)
At the start: 0 parts

Commit message: feat: draw the main board schematic
The FeatherS3D plugs into fab-fitted sockets. The panel goes through a
reverse-polarity P-FET and the solar INA226 (0x40) to a CN3163 charging
at about 495 mA; DW01A and FS8205A protect the cell, and a second INA226
(0x41) measures everything the Feather draws. The NAU7802 follows its
datasheet application circuit, with the bridge ring joining four per-cell
terminals. CHRG and DONE reach IO5 and IO6, and 3.3k pull-ups on LDO2
replace the breakouts' ones for the hive cable.
Parts:
- added C1, C14, C2: 10u, Capacitor_SMD:C_0603_1608Metric, symbol Device:C
- added C10, C12, C13, C3, C8, C9: 100n, Capacitor_SMD:C_0603_1608Metric, symbol Device:C
- added C11: 330p, Capacitor_SMD:C_0603_1608Metric, symbol Device:C
- added C4: 470u, Capacitor_SMD:CP_Elec_6.3x7.7, symbol Device:C_Polarized
- added C5, C6: 1u, Capacitor_SMD:C_0603_1608Metric, symbol Device:C
- added H1, H2, H3, H4: MountingHole, MountingHole:MountingHole_3.2mm_M3, symbol Mechanical:MountingHole
- added J1: RJHSE5380, Connector_RJ:RJ45_Amphenol_RJHSE5380, symbol Connector:RJ45_Shielded
- added J2: FEATHER_L, Connector_PinSocket_2.54mm:PinSocket_1x16_P2.54mm_Vertical, symbol Connector:Conn_01x16_Socket
- added J3: FEATHER_R, Connector_PinSocket_2.54mm:PinSocket_1x12_P2.54mm_Vertical, symbol Connector:Conn_01x12_Socket
- added J4: SOLAR, Connector_Phoenix_MC:PhoenixContact_MC_1,5_2-G-3.5_1x02_P3.50mm_Horizontal, symbol Connector:Screw_Terminal_01x02
- added J5: BATTERY, Connector_JST:JST_PH_B2B-PH-K_1x02_P2.00mm_Vertical, symbol Connector_Generic:Conn_01x02
- added J6: CELL1, Connector_Phoenix_MC:PhoenixContact_MC_1,5_3-G-3.5_1x03_P3.50mm_Horizontal, symbol Connector:Screw_Terminal_01x03
- added J7: CELL2, Connector_Phoenix_MC:PhoenixContact_MC_1,5_3-G-3.5_1x03_P3.50mm_Horizontal, symbol Connector:Screw_Terminal_01x03
- added J8: CELL3, Connector_Phoenix_MC:PhoenixContact_MC_1,5_3-G-3.5_1x03_P3.50mm_Horizontal, symbol Connector:Screw_Terminal_01x03
- added J9: CELL4, Connector_Phoenix_MC:PhoenixContact_MC_1,5_3-G-3.5_1x03_P3.50mm_Horizontal, symbol Connector:Screw_Terminal_01x03
- added Q1: AO3401A, Package_TO_SOT_SMD:SOT-23, symbol Transistor_FET:AO3401A
- added Q2: FS8205A, Package_TO_SOT_SMD:SOT-23-6, symbol beehive:FS8205A
- added R1, R5: 0.1, Resistor_SMD:R_1206_3216Metric, symbol Device:R
- added R10, R11: 33, Resistor_SMD:R_0603_1608Metric, symbol Device:R
- added R2: 2.4k, Resistor_SMD:R_0603_1608Metric, symbol Device:R
- added R3: 100, Resistor_SMD:R_0603_1608Metric, symbol Device:R
- added R4: 1k, Resistor_SMD:R_0603_1608Metric, symbol Device:R
- added R6, R7: 47, Resistor_SMD:R_0603_1608Metric, symbol Device:R
- added R8, R9: 3.3k, Resistor_SMD:R_0603_1608Metric, symbol Device:R
- added TP1: BAT+, TestPoint:TestPoint_Pad_D1.5mm, symbol Connector:TestPoint
- added TP10: WS, TestPoint:TestPoint_Pad_D1.5mm, symbol Connector:TestPoint
- added TP11: SCK, TestPoint:TestPoint_Pad_D1.5mm, symbol Connector:TestPoint
- added TP12: SD, TestPoint:TestPoint_Pad_D1.5mm, symbol Connector:TestPoint
- added TP13: CHRG, TestPoint:TestPoint_Pad_D1.5mm, symbol Connector:TestPoint
- added TP14: DONE, TestPoint:TestPoint_Pad_D1.5mm, symbol Connector:TestPoint
- added TP15: DRDY, TestPoint:TestPoint_Pad_D1.5mm, symbol Connector:TestPoint
- added TP16: AVDD, TestPoint:TestPoint_Pad_D1.5mm, symbol Connector:TestPoint
- added TP2: BAT-, TestPoint:TestPoint_Pad_D1.5mm, symbol Connector:TestPoint
- added TP3: VBAT_F, TestPoint:TestPoint_Pad_D1.5mm, symbol Connector:TestPoint
- added TP4: SOLAR, TestPoint:TestPoint_Pad_D1.5mm, symbol Connector:TestPoint
- added TP5: CHG_IN, TestPoint:TestPoint_Pad_D1.5mm, symbol Connector:TestPoint
- added TP6: GND, TestPoint:TestPoint_Pad_D1.5mm, symbol Connector:TestPoint
- added TP7: +3V3, TestPoint:TestPoint_Pad_D1.5mm, symbol Connector:TestPoint
- added TP8: SDA, TestPoint:TestPoint_Pad_D1.5mm, symbol Connector:TestPoint
- added TP9: SCL, TestPoint:TestPoint_Pad_D1.5mm, symbol Connector:TestPoint
- added U1: INA226 (0x40), Package_SO:TSSOP-10_3x3mm_P0.5mm, symbol Sensor_Energy:INA226
- added U2: CN3163, Package_SO:SOIC-8-1EP_3.9x4.9mm_P1.27mm_EP2.41x3.3mm_ThermalVias, symbol Battery_Management:CN3163
- added U3: DW01A, Package_TO_SOT_SMD:SOT-23-6, symbol Battery_Management:DW01A
- added U4: INA226 (0x41), Package_SO:TSSOP-10_3x3mm_P0.5mm, symbol Sensor_Energy:INA226
- added U5: NAU7802, Package_SO:SOIC-16_3.9x9.9mm_P1.27mm, symbol beehive:NAU7802
Connections:
- new net +3V3: C12.1, C13.1, C14.1, C6.1, J1.5, J2.16 (Pin_16), R8.1, R9.1, TP7.1, U1.6 (VS), U4.2 (A0), U4.6 (VS), U5.15 (DVDD)
- new net AVDD: C5.1, C9.1, J6.1 (Pin_1), TP16.1, U5.1 (REFP), U5.16 (AVDD/LDO)
- new net BAT+: C2.1, J5.2 (Pin_2), R3.1, R5.1, TP1.1, U2.5 (BAT), U2.8 (FB), U4.10 (Vin+)
- new net BAT-: C3.2, J5.1 (Pin_1), Q2.1 (S1), TP2.1, U3.6 (GND)
- new net CELL_AN: J7.1 (Pin_1), R6.1
- new net CELL_AP: J9.1 (Pin_1), R7.1
- new net CHG_IN: C1.1, R1.2, TP5.1, U1.8 (Vbus), U1.9 (Vin-), U2.4 (VIN)
- new net CHRG: J2.10 (Pin_10), TP13.1, U2.7 (~{CHRG})
- new net DONE: J2.9 (Pin_9), TP14.1, U2.6 (~{DONE})
- new net DRDY: TP15.1, U5.12 (DRDY)
- new net DW_CS: R4.1, U3.2 (CS)
- new net DW_OC: Q2.4 (G2), U3.3 (OC)
- new net DW_OD: Q2.6 (G1), U3.1 (OD)
- new net DW_VCC: C3.1, R3.2, U3.5 (VCC)
- new net GND: C1.2, C12.2, C13.2, C14.2, C2.2, C4.2, C5.2, C6.2, C8.2, C9.2, J1.2, J1.6, J1.SH, J2.4 (Pin_4), J4.2 (Pin_2), J8.1 (Pin_1), Q1.1 (G), Q2.3 (S2), R2.2, R4.2, TP6.1, U1.1 (A1), U1.2 (A0), U1.7 (GND), U2.1 (TEMP), U2.3 (GND), U2.9 (GND), U4.1 (A1), U4.7 (GND), U5.7 (REFN), U5.8 (AVSS), U5.9 (DVSS)
- new net ISET: R2.1, U2.2 (ISET)
- new net PROT_D: Q2.2 (D12), Q2.5 (D12)
- new net RING_B23: J7.3 (Pin_3), J8.3 (Pin_3)
- new net RING_B41: J6.3 (Pin_3), J9.3 (Pin_3)
- new net RING_W12: J6.2 (Pin_2), J7.2 (Pin_2)
- new net RING_W34: J8.2 (Pin_2), J9.2 (Pin_2)
- new net SCK: J1.1, R11.2, TP11.1
- new net SCK_F: J3.6 (Pin_6), R11.1
- new net SCL: J1.3, J3.2 (Pin_2), R9.2, TP9.1, U1.5 (SCL), U4.5 (SCL), U5.13 (SCLK)
- new net SD: J1.8, J3.7 (Pin_7), TP12.1
- new net SDA: J1.4, J3.1 (Pin_1), R8.2, TP8.1, U1.4 (SDA), U4.4 (SDA), U5.14 (SDIO)
- new net SOLAR: Q1.2 (S), R1.1, TP4.1, U1.10 (Vin+)
- new net SOLAR_RAW: J4.1 (Pin_1), Q1.3 (D)
- new net VBAT_F: C4.1, J3.12 (Pin_12), R5.2, TP3.1, U4.8 (Vbus), U4.9 (Vin-)
- new net VBG: C8.1, U5.6 (VBG)
- new net VIN1N: C10.2, R6.2, U5.2 (VIN1N)
- new net VIN1P: C10.1, R7.2, U5.3 (VIN1P)
- new net VIN2N: C11.2, U5.4 (VIN2N)
- new net VIN2P: C11.1, U5.5 (VIN2P)
- new net WS: J1.7, R10.2, TP10.1
- new net WS_F: J3.5 (Pin_5), R10.1
- no-connect marks 0 -> 23
Other:
- note added: "FeatherS3D on female headers (Unexpected Maker pinout card) J2, USB-end row: 1 RST, 2 3V3, 3 IO0, 4 GND, 5 IO17, 6 IO18, 7 IO14, 8 IO12, 9 IO6 (DONE), 10 IO5 (CHRG), 11 IO36, 12 IO35, 13 IO37, 14 IO44/RX, 15 IO43/TX, 16 LDO2 (+3V3) J3, opposite row: 1 IO8/SDA, 2 IO9/SCL, 3 IO33, 4 IO38, 5 IO1 (WS), 6 IO3 (SCK), 7 IO7 (SD), 8 IO10, 9 IO11, 10 5V, 11 EN, 12 VBAT J3 pin 1 sits opposite J2 pin 16; J3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"

Commit message: fix: act on the schematic review
The I2C pull-ups move to the Feather's always-on 3V3 so they no longer
feed the sensor rail during deep sleep. Both boards get SRV05-4 ESD
arrays on every hive cable line, with VP open so the steering diodes
cannot back-power the rail either. The microphone drives the cable
through 33 Ω, the charger input capacitor is now 25 V, and the battery
connector's value names its polarity.
Parts:
- added U6, U7: SRV05-4, Package_TO_SOT_SMD:SOT-23-6, symbol Power_Protection:SRV05-4
- C1: value 10u -> 10u 25V; LCSC C19702 -> C96446
- J5: value BATTERY -> BATTERY (1 -, 2 +)
Connections:
- net +3V3: now also U7.3 (IO2); no longer R8.1, R9.1
- net GND: now also U6.2 (VN), U7.2 (VN)
- net SCK: now also U6.6 (IO4)
- net SCL: now also U6.3 (IO2)
- net SD: now also U7.1 (IO1)
- net SDA: now also U6.1 (IO1)
- net WS: now also U6.4 (IO3)
- net 3V3_AON: now reaches J2.2 (Pin_2)
- net 3V3_AON: now also R8.1, R9.1
- no-connect marks 23 -> 26
Other:
- note added: "Hive cable ESD: VP left open so the steering diodes cannot back-power +3V3 while LDO2 is off."
- note added: "I2C pull-ups on the Feather's always-on 3V3 so they cannot feed the sensor rail while LDO2 is off."

Commit message: feat: charge with a BQ24210 instead of the CN3163
The panel measured 7.18 V unloaded, above the CN3163's 6.5 V absolute
maximum, and it sits unloaded whenever the cell is full. The BQ24210 is
rated to 20 V with an over-voltage cut-off, holds the panel at 5.0 V and
runs in its solar limited-power mode. Its CHG and PG outputs replace
CHRG and DONE on IO5 and IO6.
Parts:
- removed U2: CN3163, Package_SO:SOIC-8-1EP_3.9x4.9mm_P1.27mm_EP2.41x3.3mm_ThermalVias, symbol Battery_Management:CN3163
- added R12, R13: 10k, Resistor_SMD:R_0603_1608Metric, symbol Device:R
- added U2: BQ24210, Package_SON:WSON-10-1EP_2x3mm_P0.5mm_EP0.84x2.4mm_ThermalVias, symbol beehive:BQ24210
- R2: value 2.4k -> 820; LCSC C22940 -> C23253
- TP13: value CHRG -> CHG
- TP14: value DONE -> PG
Connections:
- net BAT+: now also U2.10 (BAT)
- net CHG_IN: now also U2.1 (VBUS)
- net GND: now also R12.2, U2.11 (EP), U2.3 (VSS), U2.7 (EN)
- net ISET: now also U2.2 (ISET)
- net CHRG renamed CHG
- net CHG: now also U2.8 (~{CHG})
- net DONE renamed PG
- net PG: now also U2.6 (~{PG})
- new net BQ_TS: R13.1, U2.5 (TS)
- new net VDPM: R12.1, U2.9 (VDPM)
- new net VTSB: R13.2, U2.4 (VTSB)

Commit message: fix: use JLCPCB-drillable and exact footprints
The BQ24210's thermal-via footprint drills 0.2 mm, below JLCPCB's 0.3 mm standard; vias go in at layout instead. The INA226s use MSOP-10, TI's DGS land pattern, rather than TSSOP-10.
Parts:
- U1, U4: footprint Package_SO:TSSOP-10_3x3mm_P0.5mm -> Package_SO:MSOP-10_3x3mm_P0.5mm
- U2: footprint Package_SON:WSON-10-1EP_2x3mm_P0.5mm_EP0.84x2.4mm_ThermalVias -> Package_SON:WSON-10-1EP_2x3mm_P0.5mm_EP0.84x2.4mm
Changed lines of the file:
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@@
 			)
 		)
-		(property "Footprint" "Package_SO:TSSOP-10_3x3mm_P0.5mm"
+		(property "Footprint" "Package_SO:MSOP-10_3x3mm_P0.5mm"
 			(at 96.52 88.9 0)
 			(hide yes)
@@
 			)
 		)
-		(property "Footprint" "Package_SO:TSSOP-10_3x3mm_P0.5mm"
+		(property "Footprint" "Package_SO:MSOP-10_3x3mm_P0.5mm"
 			(at 312.42 88.9 0)
 			(hide yes)
@@
 			)
 		)
-		(property "Footprint" "Package_SON:WSON-10-1EP_2x3mm_P0.5mm_EP0.84x2.4mm_ThermalVias"
+		(property "Footprint" "Package_SON:WSON-10-1EP_2x3mm_P0.5mm_EP0.84x2.4mm"
 			(at 154.94 55.88 0)
 			(hide yes)
